Commit message: add inertia sphere and cylinder, add collision robot

File: src/my_robot_description/urdf/common_properties.xacro (robot description, xacro)
@@ -18,3 +18,25 @@
         </inertial>
     </xacro:macro>
+    <!-- wheel right/left inertia -->
+     <xacro:macro name="cylinder_inertia" params="m l r xyz rpy">
+        <inertial>
+            <origin xyz="${xyz}" rpy="${rpy}" />
+            <mass value="${m}" />
+            <inertia ixx="${(m/12) * (3*r*r + l*l)}" ixy="0" ixz="0"
+                     iyy="${(m/12) * (3*r*r + l*l)}" iyz="0"
+                     izz="${(m/2) * r*r}"
+            />
+        </inertial>
+     </xacro:macro>
+     <!-- caster wheel inertia -->
+      <xacro:macro name="sphere_inertia" params="m r xyz rpy">
+        <inertial>
+            <origin xyz="${xyz}" rpy="${rpy}" />
+            <mass value="${m}" />
+            <inertia ixx="${(2/5) * m * r*r}" ixy="0" ixz="0"
+                     iyy="${(2/5) * m * r*r}" iyz="0"
+                     izz="${(2/5) * m * r*r}"
+            />
+        </inertial>
+      </xacro:macro>
 </robot>

File: src/my_robot_description/urdf/mobile_base.xacro (robot description, xacro)
@@ -14,4 +14,11 @@
             <material name="green" />
         </visual>
+        <collision>
+            <geometry>
+                <box size="${base_length} ${base_width} ${base_height}" /> <!--length width height-->
+            </geometry>
+            <origin xyz="0 0 ${base_height / 2.0}" rpy="0 0 0"></origin> <!-- roll pitch yaw -->
+            <material name="green" />
+        </collision>
         <xacro:box_inertia m="5.0" l="${base_length}" w="${base_width}" h="${base_height}"
                            xyz="0 0 ${base_height / 2.0}" rpy="0 0 0" />
@@ -26,4 +33,13 @@
                 <material name="grey" />
             </visual>
+            <collision>
+                <geometry>
+                    <cylinder radius="${wheel_radius}" length="${wheel_length}" />
+                </geometry>
+                <origin xyz="0 0 0" rpy="${pi / 2.0} 0 0" />
+                <material name="grey" />
+            </collision>
+            <xacro:cylinder_inertia m="1.0" l="${wheel_length}" r="${wheel_radius}"
+                                 xyz="0 0 0" rpy="${pi / 2.0} 0 0" />
         </link>
     </xacro:macro>
@@ -46,9 +62,17 @@
         <visual>
             <geometry>
-                <sphere radius="0.05" />
+                <sphere radius="${wheel_radius / 2.0}" />
             </geometry>
             <origin xyz="0 0 0" rpy="0 0 0" />
             <material name="grey" />
         </visual>
+        <collision>
+            <geometry>
+                <sphere radius="${wheel_radius / 2.0}" />
+            </geometry>
+            <origin xyz="0 0 0" rpy="0 0 0" />
+            <material name="grey" />
+        </collision>
+        <xacro:sphere_inertia m="0.5" r="${wheel_radius / 2.0}" xyz=" 0 0 0" rpy="0 0 0" />
      </link>
      <joint name="base_caster_wheel_joint" type="continuous">
